Commit message: feat(system): 接入双踝编码器解析、标定与录包链路
兼容0x15基础帧并解析LEN=68双踝紧凑尾部，校验节点、有效性与陈旧状态；导出左右踝位置、滤波角速度和原始诊断接口，驱动JointState与RViz显示；增加机械零偏、方向配置及只读圆周均值标定工具；将踝关节和原始状态纳入录包前内容检查，补充操作与安全说明；新增LEN=68、旧LEN=42兼容和跨零点修正回归测试。

File: src/exoskeleton_hardware/urdf/exo_ros2_control.urdf.xacro (robot description, xacro)
@@ -362,5 +362,5 @@
   <joint
     name="left_ankle"
-    type="fixed">
+    type="revolute">
     <origin
       xyz="0.345999999999997 0.000100000000003042 0.017"
@@ -370,4 +370,6 @@
     <child
       link="left_foot" />
+    <axis xyz="0 0 1" />
+    <limit lower="-0.5236" upper="0.5236" effort="0" velocity="10" />
   </joint>
   <link
@@ -682,5 +684,5 @@
   <joint
     name="right_ankle"
-    type="fixed">
+    type="revolute">
     <origin
       xyz="0.346000000000043 9.99999997232381E-05 -0.0170000000012193"
@@ -690,4 +692,6 @@
     <child
       link="right_foot_link" />
+    <axis xyz="0 0 -1" />
+    <limit lower="-0.5236" upper="0.5236" effort="0" velocity="10" />
   </joint>
 <ros2_control name="ExoskeletonSystem" type="system">
@@ -702,4 +706,6 @@
       <param name="torque_limit">200.0</param>
       <param name="current_limit">20.0</param>
+      <!-- 踝角速度由上位机差分后一阶低通；(0,1]，越小滤波越强 -->
+      <param name="ankle_velocity_filter_alpha">0.2</param>
       <!-- 真机测试: false 打开串口; 无硬件调试时改回 true 跳过串口 -->
       <param name="use_mock">false</param>
@@ -762,4 +768,21 @@
       <state_interface name="feedback_sequence"/>
     </joint>
+    <!-- 被动踝关节只导出状态，无 command interface，不会使能或施加力矩。 -->
+    <sensor name="left_ankle">
+      <state_interface name="position"/>
+      <state_interface name="velocity"/>
+      <state_interface name="raw_count"/>
+      <state_interface name="node_id"/>
+      <state_interface name="feedback_valid"/>
+      <state_interface name="stale"/>
+    </sensor>
+    <sensor name="right_ankle">
+      <state_interface name="position"/>
+      <state_interface name="velocity"/>
+      <state_interface name="raw_count"/>
+      <state_interface name="node_id"/>
+      <state_interface name="feedback_valid"/>
+      <state_interface name="stale"/>
+    </sensor>
   </ros2_control>
 </robot>
